File: open-control-board-hv.kicad_sch (KiCad schematic)
At the start: 20 parts, among them J3 TE 160650-2, J4 TE 160650-2, J5 TE 160650-2, J6 TE 160650-2, J7 TE 160650-2, J8 TE 160650-2, K1 RT314A12, U11 ALDP112, U12 ALDP112, U13 ALDP112

Commit message: Updated with manufacturing data and switched footprint for fastons
Parts:
- J3, J4, J5, J6, J7, J8: footprint 1289:KEYSTONE_1289 -> 624091:TE_62409-1
Changed lines of the file:
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@@
       (effects (font (size 1.27 1.27)))
     )
-    (property "Footprint" "1289:KEYSTONE_1289" (at 200.66 92.71 0)
+    (property "Footprint" "624091:TE_62409-1" (at 200.66 92.71 0)
       (effects (font (size 1.27 1.27)) hide)
     )
@@
       (effects (font (size 1.27 1.27)))
     )
-    (property "Footprint" "1289:KEYSTONE_1289" (at 36.83 85.09 0)
+    (property "Footprint" "624091:TE_62409-1" (at 36.83 85.09 0)
       (effects (font (size 1.27 1.27)) hide)
     )
@@
       (effects (font (size 1.27 1.27)) (justify left))
     )
-    (property "Footprint" "1289:KEYSTONE_1289" (at 82.55 135.89 0)
+    (property "Footprint" "624091:TE_62409-1" (at 82.55 135.89 0)
       (effects (font (size 1.27 1.27)) hide)
     )
@@
       (effects (font (size 1.27 1.27)))
     )
-    (property "Footprint" "1289:KEYSTONE_1289" (at 36.83 93.98 0)
+    (property "Footprint" "624091:TE_62409-1" (at 36.83 93.98 0)
       (effects (font (size 1.27 1.27)) hide)
     )
@@
       (effects (font (size 1.27 1.27)))
     )
-    (property "Footprint" "1289:KEYSTONE_1289" (at 199.39 22.86 0)
+    (property "Footprint" "624091:TE_62409-1" (at 199.39 22.86 0)
       (effects (font (size 1.27 1.27)) hide)
     )
@@
       (effects (font (size 1.27 1.27)))
     )
-    (property "Footprint" "1289:KEYSTONE_1289" (at 201.93 160.02 0)
-      (effects (font (size 1.27 1.27)) hide)
-    )
+    (property "Footprint" "624091:TE_62409-1" (at 201.93 160.02 0)
+      (effects (font (size 1.27 1.27)) hide)
+    )

Commit message: Cleanup
Parts:
- removed U11, U12, U13: ALDP112, ALDP112:PAN_ALD_PAN, symbol ALDP112:ALDP112
- added K2, K3, K4: ALDP112, ALDP112:PAN_ALD_PAN, symbol Relay:Relay_SPST-NO
- D2, D4, D5, D8, U2: Comment (none) -> Hand solder
Connections:
- net +12VA: now also K2.4, K3.4, K4.4
- net FA7_CTRL: now also D5.2 (A), K4.3; no longer D2.2 (A)
- net FA8_CTRL: now also K3.3
- net FA9_CTRL: now also D2.2 (A), K2.3; no longer D5.2 (A)
- net PH: now also K2.2, K3.2, K4.2
- net at J4.1 (Pin_1): now also K3.1
- net at J5.1 (Pin_1): now also K4.1
- net at J3.1 (Pin_1): now also K2.1
- net PH_PRE_FUSE: no longer names the net of F1.1, J7.1 (Pin_1)
Other:
- note added: "16A Relay (230VAC, 12VDC)"
- note added: "5A Relays (230VAC, 12VDC)"
- note added: "AC/DC converter (230VAC, 12VDC)"
- note added: "Main board connector (12VDC)"
- note added: "Power connector (230VAC)"
- moved on the sheet: D4, D8, H1, H2, H3, J4, J6, J7, J8, JP1, K1, U2

Commit message: R0C
Connections:
- net PH: now also F1.1, J7.1 (Pin_1), K1.12; no longer F1.2, U2.2 (ACL)
- new net PH_FUSED: F1.2, U2.2 (ACL)
- no-connect marks 1 -> 0
Other:
- moved on the sheet: F1
Changed lines of the file:
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@@
 (kicad_sch (version 20230121) (generator eeschema)
   (paper "A3")
+  (junction (at 101.6 27.94) (diameter 0) (color 0 0 0 0)
+  )
   (junction (at 121.92 173.99) (diameter 0) (color 0 0 0 0)
   )
@@
   (junction (at 120.65 129.54) (diameter 0) (color 0 0 0 0)
   )
-  (no_connect (at 60.96 105.41))
   (wire (pts (xy 138.43 82.55) (xy 140.97 82.55))
     (stroke (width 0) (type default))
@@
     (stroke (width 0) (type default))
   )
-  (wire (pts (xy 96.52 27.94) (xy 91.44 27.94))
+  (wire (pts (xy 104.14 27.94) (xy 101.6 27.94))
     (stroke (width 0) (type default))
   )
@@
     (stroke (width 0) (type default))
   )
+  (wire (pts (xy 101.6 27.94) (xy 91.44 27.94))
+    (stroke (width 0) (type default))
+  )
   (wire (pts (xy 31.75 35.56) (xy 43.18 35.56))
     (stroke (width 0) (type default))
@@
     (stroke (width 0) (type default))
   )
+  (wire (pts (xy 101.6 22.86) (xy 101.6 27.94))
+    (stroke (width 0) (type default))
+  )
   (wire (pts (xy 31.75 27.94) (xy 43.18 27.94))
     (stroke (width 0) (type default))
@@
     (stroke (width 0) (type default))
   )
-  (wire (pts (xy 104.14 27.94) (xy 110.49 27.94))
+  (wire (pts (xy 111.76 27.94) (xy 118.11 27.94))
     (stroke (width 0) (type default))
   )
@@
     )
   )
+  (global_label "PH" (shape passive) (at 101.6 22.86 90) (fields_autoplaced)
+    (effects (font (size 1.27 1.27)) (justify left))
+    (property "Intersheetrefs" "${INTERSHEET_REFS}" (at 101.6 18.3856 90)
+      (effects (font (size 1.27 1.27)) (justify left) hide)
+    )
+  )
   (global_label "PH" (shape passive) (at 138.43 163.83 0) (fields_autoplaced)
     (effects (font (size 1.27 1.27)) (justify left))
     (property "Intersheetrefs" "${INTERSHEET_REFS}" (at 142.9044 163.83 0)
-      (effects (font (size 1.27 1.27)) (justify left) hide)
-    )
-  )
-  (global_label "PH" (shape passive) (at 110.49 27.94 0) (fields_autoplaced)
-    (effects (font (size 1.27 1.27)) (justify left))
-    (property "Intersheetrefs" "${INTERSHEET_REFS}" (at 114.9644 27.94 0)
       (effects (font (size 1.27 1.27)) (justify left) hide)
     )
@@
     )
   )
+  (global_label "PH_FUSED" (shape passive) (at 118.11 27.94 270) (fields_autoplaced)
+    (effects (font (size 1.27 1.27)) (justify right))
+    (property "Intersheetrefs" "${INTERSHEET_REFS}" (at 118.11 39.4296 90)
+      (effects (font (size 1.27 1.27)) (justify right) hide)
+    )
+  )
   (global_label "PH" (shape passive) (at 138.43 119.38 0) (fields_autoplaced)
     (effects (font (size 1.27 1.27)) (justify left))
@@
     )
   )
-  (global_label "PH" (shape passive) (at 33.02 64.77 180) (fields_autoplaced)
+  (global_label "PH_FUSED" (shape passive) (at 33.02 64.77 180) (fields_autoplaced)
     (effects (font (size 1.27 1.27)) (justify right))
-    (property "Intersheetrefs" "${INTERSHEET_REFS}" (at 28.5456 64.77 0)
+    (property "Intersheetrefs" "${INTERSHEET_REFS}" (at 21.5304 64.77 0)
       (effects (font (size 1.27 1.27)) (justify right) hide)
+    )
+  )
+  (global_label "PH" (shape passive) (at 60.96 105.41 90) (fields_autoplaced)
+    (effects (font (size 1.27 1.27)) (justify left))
+    (property "Intersheetrefs" "${INTERSHEET_REFS}" (at 60.96 100.9356 90)
+      (effects (font (size 1.27 1.27)) (justify left) hide)
     )
   )
@@
   (netclass_flag "" (length 2.54) (shape round) (at 93.98 27.94 0) (fields_autoplaced)
     (effects (font (size 1.27 1.27)) (justify left bottom))
-    (property "Netclass" "230V" (at 94.6785 25.4 0)
+    (property "Netclass" "230V_16A" (at 94.6785 25.4 0)
       (effects (font (size 1.27 1.27) italic) (justify left))
     )
@@
   (netclass_flag "" (length 2.54) (shape round) (at 66.04 102.87 90) (fields_autoplaced)
     (effects (font (size 1.27 1.27)) (justify left bottom))
-    (property "Netclass" "230V" (at 63.5 102.1715 90)
+    (property "Netclass" "230V_16A" (at 63.5 102.1715 90)
       (effects (font (size 1.27 1.27) italic) (justify left))
     )
@@
   (netclass_flag "" (length 2.54) (shape round) (at 119.38 161.29 0) (fields_autoplaced)
     (effects (font (size 1.27 1.27)) (justify left bottom))
-    (property "Netclass" "230V" (at 120.0785 158.75 0)
+    (property "Netclass" "230V_5A" (at 120.0785 158.75 0)
       (effects (font (size 1.27 1.27) italic) (justify left))
     )
@@
   (netclass_flag "" (length 2.54) (shape round) (at 119.38 69.85 180) (fields_autoplaced)
     (effects (font (size 1.27 1.27)) (justify right bottom))
-    (property "Netclass" "230V" (at 120.0785 72.39 0)
+    (property "Netclass" "230V_5A" (at 120.0785 72.39 0)
       (effects (font (size 1.27 1.27) italic) (justify left))
     )
@@
     )
   )
-  (netclass_flag "" (length 2.54) (shape round) (at 106.68 27.94 0) (fields_autoplaced)
-    (effects (font (size 1.27 1.27)) (justify left bottom))
-    (property "Netclass" "230V" (at 107.3785 25.4 0)
+  (netclass_flag "" (length 2.54) (shape round) (at 114.3 27.94 0) (fields_autoplaced)
+    (effects (font (size 1.27 1.27)) (justify left bottom))
+    (property "Netclass" "230V_500MA" (at 114.9985 25.4 0)
       (effects (font (size 1.27 1.27) italic) (justify left))
     )
@@
   (netclass_flag "" (length 2.54) (shape round) (at 93.98 40.64 0) (fields_autoplaced)
     (effects (font (size 1.27 1.27)) (justify left bottom))
-    (property "Netclass" "230V" (at 94.6785 38.1 0)
+    (property "Netclass" "230V_16A" (at 94.6785 38.1 0)
       (effects (font (size 1.27 1.27) italic) (justify left))
     )
@@
   (netclass_flag "" (length 2.54) (shape round) (at 119.38 116.84 0) (fields_autoplaced)
     (effects (font (size 1.27 1.27)) (justify left bottom))
-    (property "Netclass" "230V" (at 120.0785 114.3 0)
+    (property "Netclass" "230V_5A" (at 120.0785 114.3 0)
       (effects (font (size 1.27 1.27) italic) (justify left))
     )
@@
     )
   )
-  (symbol (lib_id "Device:Fuse") (at 100.33 27.94 90) (unit 1)
+  (symbol (lib_id "Device:Fuse") (at 107.95 27.94 90) (unit 1)
     (in_bom yes) (on_board yes) (dnp no)
-    (property "Reference" "F1" (at 100.33 22.86 90)
-      (effects (font (size 1.27 1.27)))
-    )
-    (property "Value" "Schurter FRT 250T 7100.1009.13" (at 91.44 31.75 90)
-      (effects (font (size 1.27 1.27)))
-    )
-    (property "Footprint" "1289:FRT 250T" (at 100.33 29.718 90)
-      (effects (font (size 1.27 1.27)) hide)
-    )
-    (property "Datasheet" "~" (at 100.33 27.94 0)
-      (effects (font (size 1.27 1.27)) hide)
-    )
-    (property "Comment" "Hand solder" (at 100.33 27.94 0)
-      (effects (font (size 1.27 1.27)) hide)
-    )
-    (property "Digikey" "https://www.digikey.se/en/products/detail/schurter-inc/7100-1009-13/639906" (at 100.33 27.94 0)
-      (effects (font (size 1.27 1.27)) hide)
-    )
+    (property "Reference" "F1" (at 107.95 22.86 90)
+      (effects (font (size 1.27 1.27)))
+    )
+    (property "Value" "Schurter FRT 250T 7100.1009.13" (at 99.06 31.75 90)
+      (effects (font (size 1.27 1.27)))
+    )
+    (property "Footprint" "1289:FRT 250T" (at 107.95 29.718 90)
+      (effects (font (size 1.27 1.27)) hide)
+    )
+    (property "Datasheet" "~" (at 107.95 27.94 0)
+      (effects (font (size 1.27 1.27)) hide)
+    )
+    (property "Comment" "Hand solder" (at 107.95 27.94 0)
+      (effects (font (size 1.27 1.27)) hide)
+    )
+    (property "Digikey" "https://www.digikey.se/en/products/detail/schurter-inc/7100-1009-13/639906" (at 107.95 27.94 0)
+      (effects (font (size 1.27 1.27)) hide)
+    )
